File: ESP32_Tracker.kicad_sch (KiCad schematic)
At the start: 61 parts, among them J1 USB_C_Receptacle_USB2.0_16P, J2 Conn_01x02_Socket, J3 Micro_SD_Card_Det1, SW1 SW_Push, SW2 SW_Push, SW3 SW_Push, U1 XC6220B331MR-G, U2 USBLC6-2SC6, U3 MP2667, U4 SAM-M10Q, U5 LIS2MDL, U6 ESP32-S3-MINI-1

Commit message: initial board layout completed
Parts:
- removed C1, C15, C4, C5, C9: 10u, Capacitor_SMD:C_0805_2012Metric, symbol Device:C
- removed C10, C11, C13, C14, C18, C6, C8: 0.1u, Capacitor_SMD:C_0805_2012Metric, symbol Device:C
- removed C12: 22u, Capacitor_SMD:C_0805_2012Metric, symbol Device:C
- removed C16, C2: 1u, Capacitor_SMD:C_0805_2012Metric, symbol Device:C
- removed C17: 0.22u, Capacitor_SMD:C_0805_2012Metric, symbol Device:C
- removed C3, C7: 2.2u, Capacitor_SMD:C_0805_2012Metric, symbol Device:C
- removed D1: LED, LED_SMD:LED_0805_2012Metric, symbol Device:LED
- removed J1: USB_C_Receptacle_USB2.0_16P, Connector_USB:USB_C_Receptacle_G-Switch_GT-USB-7010ASV, symbol Connector:USB_C_Receptacle_USB2.0_16P
- removed J2: Conn_01x02_Socket, Connector_JST:JST_PH_S2B-PH-K_1x02_P2.00mm_Horizontal, symbol Connector:Conn_01x02_Socket
- removed J3: Micro_SD_Card_Det1, MSD-4-A_DL:CUI_MSD-4-A, symbol Connector:Micro_SD_Card_Det1
- removed R1, R3: 5.1k, Resistor_SMD:R_0805_2012Metric, symbol Device:R_US
- removed R10, R11, R12, R13, R14, R15, R16, R18, R2, R4, R8, R9: 10k, Resistor_SMD:R_0805_2012Metric, symbol Device:R_US
- removed R17, R6, R7: 2.2k, Resistor_SMD:R_0805_2012Metric, symbol Device:R_US
- removed R5: 100k, Resistor_SMD:R_0805_2012Metric, symbol Device:R_US
- removed SW1, SW2, SW3: SW_Push, Button_Switch_SMD:SW_SPST_TS-1088-xR020, symbol Switch:SW_Push
- removed TP1, TP2, TP3, TP4, TP5, TP6, TP7, TP8: TestPoint, TestPoint:TestPoint_Pad_D1.5mm, symbol Connector:TestPoint
- removed U1: XC6220B331MR-G, Package_TO_SOT_SMD:SOT-23-5, symbol Regulator_Linear:XC6220B331MR
- removed U2: USBLC6-2SC6, Package_TO_SOT_SMD:SOT-23-6, symbol Power_Protection:USBLC6-2SC6
- removed U3: MP2667, MP2667_DL:QFN-10_2MMx2MM_MNP, symbol Power_Management_MPS:MP2667
- removed U4: SAM-M10Q, RF_GPS:ublox_SAM-M8Q, symbol RF_GPS:SAM-M8Q
- removed U5: LIS2MDL, Package_LGA:LGA-12_2x2mm_P0.5mm, symbol Sensor_Magnetic:LIS2MDL
- removed U6: ESP32-S3-MINI-1, RF_Module:ESP32-S2-MINI-1, symbol RF_Module:ESP32-S3-MINI-1
- renumbered H3 to H2, H2 to H3
Connections:
- no-connect marks 32 -> 0
Other:
- added sheet MCU/PWR (MAIN.kicad_sch)
- added sheet Peripherals (peripherals.kicad_sch)
- added sheet Sensors (sensors.kicad_sch)
- note added: "ESP32 - MAX: 340mA TYP: 15-100mA (dpnd on speed/cores) GPS - MAX: 13mA TYP: 10mA MAG - MAX: 200uA TYP: 200uA SD - MAX: 50-100mA? TYP: 50-100mA OLED - MAX: 75mA TYP: 50mA TOTAL: 500mA max, 250 (high side average)"
- note added: "MAG/GPS using I2C"
- note added: "USB-C (DONE) LDO (DONE) GPS (DONE) MAGNETOMETER (DONE) MICROSD (DONE) BATTERY MGMT. (DONE) BUTTONS (DONE) STATUS LEDs (DONE) Low PWR mode (DONE) OLED CONN (DONE) PWR CONSUMPTION (IN PROGRESS)"
- note removed: "(4.5, 5, 5.5)V"
- note removed: "3.7V 2Ah LiPo"
- note removed: "5v -> 3.3v @ 1A 60mV @ 300mA"
- note removed: "BOOT"
- note removed: "Batt IC Alternatives: MP2667 MCP73871"
- note removed: "Charging IC + PWR Path Programmable charge current"
- note removed: "HIGH for I2C"
- note removed: "POLARITY OF JST?"
- note removed: "RESET"
- note removed: "Reset button? clears GNSS data and config stored in BBR"
- note removed: "USB-C (DONE) LDO (DONE) GPS (DONE) MAGNETOMETER (DONE) MICROSD (DONE) BATTERY MGMT. (DONE) BUTTONS (IN PROGRESS) STATUS LEDs (IN PROGRESS) PWR CONSUMPTION (IN PROGRESS) OLED CONN (?) RTC for Low PWR mode (Shipping mode on MP2667?)"
- note removed: "Why LiPo? Thin, compact Adafruit protection circuitry right voltage not great lifespan compared to others"
- note removed: "adafruit LiPo has built in protection circuitry only need charging IC"
- note removed: "alum."
- note removed: "bypass caps TYP.APP."
- note removed: "bypass caps typ. app."
- note removed: "ceram."
- note removed: "have primary LiPo act as backup? or add small coincell?"
- note removed: "logging on/off"
- note removed: "status LED"
- note removed: "sys load"
- note removed: "timepulse LED?"
- note removed: "toggle button record button low power"
- note removed: "typ. app."
- moved on the sheet: H1, H2, H3, H4
