File: ESP32_Tracker.kicad_pcb (KiCad board)
At the start: 4 copper layers, 60 x 75 mm, 75 parts, among them J2 Conn_01x02_Socket, J3 Conn_01x03, J4 MSD-4-A, J5 Conn_01x07_Socket, J6 USB_C_Receptacle_USB2.0_16P, SW1 SW_Push, SW2 SW_Push, SW3 SW_Push, SW4 SW_Push, SW5 SW_Push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

Commit message: modified battery terminal
Parts:
- moved C14 8.57 mm to (139.0, 100.0), turned to -90 degrees
- moved C13 4.43 mm to (130.5, 100.5), turned to 90 degrees
- moved R15 3.17 mm to (137.6, 103.0), turned to 0 degrees
Connections:
- J2 pad 1: GND -> +BATT
- J2 pad 2: +BATT -> GND
Routing:
- net +3.3V: track 59.2 -> 62.4 mm, vias 33 -> 32
- net /MCU/PWR/GPS/MAG_CLK: track 47.7 -> 50.6 mm
- net +BATT: track 21.1 -> 19.4 mm
- net GND: track 121.4 -> 120.0 mm, vias 217 -> 220
- net /MCU/PWR/GPS/MAG_DATA: track 52.3 -> 53.6 mm
Other:
- board text added: "+"
- board text added: "-"
- board text added: "MY NAME REV 1.0 1/16/2026 CLASS #"
- board text removed: "Matthew Tubbin REV 1.0 1/16/2026 ECE-212"
