File: peripherals.kicad_sch (KiCad schematic)
At the start: 12 parts, among them J4 MSD-4-A, J5 Conn_01x08_Socket

Commit message: REV 1.0 Ordered
Parts:
- renumbered C19 to C20, C20 to C21, C21 to C22, C22 to C23, J5 to J4, J4 to J5
Changed lines of the file:
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@@
 		(on_board yes)
 		(dnp no)
-		(property "Reference" "C19"
+		(property "Reference" "C20"
 			(at 109.22 126.9999 0)
 			(effects
@@
 			(project "ESP32_Tracker"
 				(path "/92195c42-0bc4-473e-a890-6f85786d3c69/397d7a99-8f38-42c5-a73f-5d1ccdc57b5a"
-					(reference "C19")
+					(reference "C20")
 					(unit 1)
 				)
@@
 		(on_board yes)
 		(dnp no)
-		(property "Reference" "C21"
+		(property "Reference" "C22"
 			(at 151.13 39.3699 0)
 			(effects
@@
 			(project "ESP32_Tracker"
 				(path "/92195c42-0bc4-473e-a890-6f85786d3c69/397d7a99-8f38-42c5-a73f-5d1ccdc57b5a"
-					(reference "C21")
+					(reference "C22")
 					(unit 1)
 				)
@@
 		(on_board yes)
 		(dnp no)
-		(property "Reference" "C20"
+		(property "Reference" "C21"
 			(at 119.38 126.9999 0)
 			(effects
@@
 			(project "ESP32_Tracker"
 				(path "/92195c42-0bc4-473e-a890-6f85786d3c69/397d7a99-8f38-42c5-a73f-5d1ccdc57b5a"
-					(reference "C20")
+					(reference "C21")
 					(unit 1)
 				)
@@
 		(dnp no)
 		(fields_autoplaced yes)
-		(property "Reference" "#PWR037"
+		(property "Reference" "#PWR039"
 			(at 137.16 125.73 0)
 			(effects
@@
 			(project "ESP32_Tracker"
 				(path "/92195c42-0bc4-473e-a890-6f85786d3c69/397d7a99-8f38-42c5-a73f-5d1ccdc57b5a"
-					(reference "#PWR037")
+					(reference "#PWR039")
 					(unit 1)
 				)
@@
 		(on_board yes)
 		(dnp no)
-		(property "Reference" "#PWR039"
+		(property "Reference" "#PWR041"
 			(at 158.75 53.34 0)
 			(effects
@@
 			(project "ESP32_Tracker"
 				(path "/92195c42-0bc4-473e-a890-6f85786d3c69/397d7a99-8f38-42c5-a73f-5d1ccdc57b5a"
-					(reference "#PWR039")
+					(reference "#PWR041")
 					(unit 1)
 				)
@@
 		(dnp no)
 		(fields_autoplaced yes)
-		(property "Reference" "#PWR040"
+		(property "Reference" "#PWR042"
 			(at 162.56 102.87 0)
 			(effects
@@
 			(project "ESP32_Tracker"
 				(path "/92195c42-0bc4-473e-a890-6f85786d3c69/397d7a99-8f38-42c5-a73f-5d1ccdc57b5a"
-					(reference "#PWR040")
+					(reference "#PWR042")
 					(unit 1)
 				)
@@
 		(dnp no)
 		(fields_autoplaced yes)
-		(property "Reference" "J5"
+		(property "Reference" "J4"
 			(at 154.94 142.2399 0)
 			(effects
@@
 			(project "ESP32_Tracker"
 				(path "/92195c42-0bc4-473e-a890-6f85786d3c69/397d7a99-8f38-42c5-a73f-5d1ccdc57b5a"
-					(reference "J5")
+					(reference "J4")
 					(unit 1)
 				)
@@
 		(on_board yes)
 		(dnp no)
-		(property "Reference" "#PWR036"
+		(property "Reference" "#PWR038"
 			(at 113.03 142.24 0)
 			(effects
@@
 			(project "ESP32_Tracker"
 				(path "/92195c42-0bc4-473e-a890-6f85786d3c69/397d7a99-8f38-42c5-a73f-5d1ccdc57b5a"
-					(reference "#PWR036")
+					(reference "#PWR038")
 					(unit 1)
 				)
@@
 		(dnp no)
 		(fields_autoplaced yes)
-		(property "Reference" "J4"
+		(property "Reference" "J5"
 			(at 193.04 72.3899 0)
 			(effects
@@
 			(project ""
 				(path "/92195c42-0bc4-473e-a890-6f85786d3c69/397d7a99-8f38-42c5-a73f-5d1ccdc57b5a"
-					(reference "J4")
+					(reference "J5")
 					(unit 1)
 				)
@@
 		(dnp no)
 		(fields_autoplaced yes)
-		(property "Reference" "#PWR038"
+		(property "Reference" "#PWR040"
 			(at 142.24 35.56 0)
 			(effects
@@
 			(project "ESP32_Tracker"
 				(path "/92195c42-0bc4-473e-a890-6f85786d3c69/397d7a99-8f38-42c5-a73f-5d1ccdc57b5a"
-					(reference "#PWR038")
+					(reference "#PWR040")
 					(unit 1)
 				)
@@
 		(on_board yes)
 		(dnp no)
-		(property "Reference" "C22"
+		(property "Reference" "C23"
 			(at 162.56 39.3699 0)
 			(effects
@@
 			(project "ESP32_Tracker"
 				(path "/92195c42-0bc4-473e-a890-6f85786d3c69/397d7a99-8f38-42c5-a73f-5d1ccdc57b5a"
-					(reference "C22")
+					(reference "C23")
 					(unit 1)
 				)
