File: sensors.kicad_sch (KiCad schematic)
At the start: 12 parts, among them U5 LIS2MDL, U6 SAM-M10Q

Commit message: Layout completed
Parts:
- C17: value 2.2u -> 10u; Distributor Link https://www.lcsc.com/product-detail/C28234.html -> https://www.lcsc.com/product-detail/C95841.html; LCSC C28234 -> C95841; MPN CL21B225KOFNNNE -> CL21B106KOQNNNE
Other:
- note added: "Potentially remove bulk cap?"
- note removed: "alum."
Changed lines of the file:
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@@
-	(text "ceram."
-		(exclude_from_sim no)
-		(at 86.868 64.262 0)
-		(effects
-			(font
-				(size 1.27 1.27)
-			)
-		)
-	)
 	(text "ceram."
 		(exclude_from_sim no)
@@
 		)
 	)
-	(text "alum."
+	(text "bypass caps\nTYP.APP.\n"
 		(exclude_from_sim no)
-		(at 61.976 64.262 0)
+		(at 76.708 51.816 0)
 		(effects
 			(font
@@
 		)
 	)
-	(text "ceram."
+	(text "Potentially remove bulk cap?\n"
 		(exclude_from_sim no)
-		(at 74.168 64.262 0)
-		(effects
-			(font
-				(size 1.27 1.27)
-			)
-		)
-	)
-	(text "bypass caps\nTYP.APP.\n"
-		(exclude_from_sim no)
-		(at 76.708 51.816 0)
+		(at 40.386 59.436 0)
 		(effects
 			(font
@@
 	)
 	(symbol
+		(lib_id "Device:C")
+		(at 168.91 59.69 0)
+		(mirror y)
+		(unit 1)
+		(exclude_from_sim no)
+		(in_bom yes)
+		(on_board yes)
+		(dnp no)
+		(property "Reference" "C17"
+			(at 165.1 58.4199 0)
+			(effects
+				(font
+					(size 1.27 1.27)
+				)
+				(justify left)
+			)
+		)
+		(property "Value" "10u"
+			(at 165.1 60.9599 0)
+			(effects
+				(font
+					(size 1.27 1.27)
+				)
+				(justify left)
+			)
+		)
+		(property "Footprint" "Capacitor_SMD:C_0805_2012Metric"
+			(at 167.9448 63.5 0)
+			(effects
+				(font
+					(size 1.27 1.27)
+				)
+				(hide yes)
+			)
+		)
+		(property "Datasheet" "https://www.lcsc.com/datasheet/C95841.pdf"
+			(at 168.91 59.69 0)
+			(effects
+				(font
+					(size 1.27 1.27)
+				)
+				(hide yes)
+			)
+		)
+		(property "Description" "Unpolarized capacitor"
+			(at 168.91 59.69 0)
+			(effects
+				(font
+					(size 1.27 1.27)
+				)
+				(hide yes)
+			)
+		)
+		(property "LCSC" "C95841"
+			(at 168.91 59.69 0)
+			(effects
+				(font
+					(size 1.27 1.27)
+				)
+				(hide yes)
+			)
+		)
+		(property "MPN" "CL21B106KOQNNNE"
+			(at 168.91 59.69 0)
+			(effects
+				(font
+					(size 1.27 1.27)
+				)
+				(hide yes)
+			)
+		)
+		(property "Manufacturer" "Samsung Electro-Mechanics"
+			(at 168.91 59.69 0)
+			(effects
+				(font
+					(size 1.27 1.27)
+				)
+				(hide yes)
+			)
+		)
+		(property "Distributor Link" "https://www.lcsc.com/product-detail/C95841.html"
+			(at 168.91 59.69 0)
+			(effects
+				(font
+					(size 1.27 1.27)
+				)
+				(hide yes)
+			)
+		)
+		(pin "2"
+		)
+		(pin "1"
+		)
+		(instances
+			(project "ESP32_Tracker"
+				(path "/92195c42-0bc4-473e-a890-6f85786d3c69/df595db4-adad-4efb-b42f-768fb30b12a2"
+					(reference "C17")
+					(unit 1)
+				)
+			)
+		)
+	)
+	(symbol
 		(lib_id "power:GND")
 		(at 96.52 101.6 0)
@@
 					(unit 1)
 				)
-			)
-		)
-	)
-	(symbol
-		(lib_id "Device:C")
-		(at 168.91 59.69 0)
-		(unit 1)
-		(exclude_from_sim no)
-		(in_bom yes)
-		(on_board yes)
-		(dnp no)
-		(property "Reference" "C17"
-			(at 161.29 59.69 90)
-			(effects
-				(font
-					(size 1.27 1.27)
-				)
-			)
-		)
-		(property "Value" "2.2u"
-			(at 163.83 59.69 90)
-			(effects
-				(font
-					(size 1.27 1.27)
-				)
-			)
-		)
-		(property "Footprint" "Capacitor_SMD:C_0805_2012Metric"
-			(at 169.8752 63.5 0)
-			(effects
-				(font
-					(size 1.27 1.27)
-				)
-				(hide yes)
-			)
-		)
-		(property "Datasheet" "https://www.lcsc.com/datasheet/C28234.pdf"
-			(at 168.91 59.69 0)
-			(effects
-				(font
-					(size 1.27 1.27)
-				)
-				(hide yes)
-			)
-		)
-		(property "Description" "Unpolarized capacitor"
-			(at 168.91 59.69 0)
-			(effects
-				(font
-					(size 1.27 1.27)
-				)
-				(hide yes)
-			)
-		)
-		(property "LCSC" "C28234"
-			(at 168.91 59.69 90)
-			(effects
-				(font
-					(size 1.27 1.27)
-				)
-				(hide yes)
-			)
-		)
-		(property "MPN" "CL21B225KOFNNNE"
-			(at 168.91 59.69 90)
-			(effects
-				(font
-					(size 1.27 1.27)
-				)
-				(hide yes)
-			)
-		)
-		(property "Manufacturer" "Samsung Electro-Mechanics"
-			(at 168.91 59.69 90)
-			(effects
-				(font
-					(size 1.27 1.27)
-				)
-				(hide yes)
-			)
-		)
-		(property "Distributor Link" "https://www.lcsc.com/product-detail/C28234.html"
-			(at 168.91 59.69 90)
-			(effects
-				(font
-					(size 1.27 1.27)
-				)
-				(hide yes)
-			)
-		)
-		(pin "2"
-		)
-		(pin "1"
-		)
-		(instances
-			(project "ESP32_Tracker"
-				(path "/92195c42-0bc4-473e-a890-6f85786d3c69/df595db4-adad-4efb-b42f-768fb30b12a2"
-					(reference "C17")
-					(unit 1)
-				)

Commit message: modified layout
Changed lines of the file:
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@@
-	)
-	(junction
-		(at 63.5 68.58)
-		(diameter 0)
-		(color 0 0 0 0)
 	)
 	(junction
@@
 	(wire
 		(pts
-			(xy 63.5 68.58) (xy 71.12 68.58)
-		)
-		(stroke
-			(width 0)
-			(type default)
-		)
-	)
-	(wire
-		(pts
 			(xy 212.09 82.55) (xy 212.09 86.36)
 		)
@@
 	(wire
 		(pts
-			(xy 71.12 77.47) (xy 71.12 68.58)
-		)
-		(stroke
-			(width 0)
-			(type default)
-		)
-	)
-	(wire
-		(pts
 			(xy 50.8 82.55) (xy 58.42 82.55)
 		)
@@
 		(pts
 			(xy 63.5 80.01) (xy 83.82 80.01)
+		)
+		(stroke
+			(width 0)
+			(type default)
+		)
+	)
+	(wire
+		(pts
+			(xy 71.12 72.39) (xy 71.12 77.47)
 		)
 		(stroke
@@
 	)
 	(symbol
+		(lib_id "power:+3.3V")
+		(at 71.12 72.39 0)
+		(unit 1)
+		(exclude_from_sim no)
+		(in_bom yes)
+		(on_board yes)
+		(dnp no)
+		(property "Reference" "#PWR04"
+			(at 71.12 76.2 0)
+			(effects
+				(font
+					(size 1.27 1.27)
+				)
+				(hide yes)
+			)
+		)
+		(property "Value" "+3.3V"
+			(at 71.12 68.326 0)
+			(effects
+				(font
+					(size 1.27 1.27)
+				)
+			)
+		)
+		(property "Footprint" ""
+			(at 71.12 72.39 0)
+			(effects
+				(font
+					(size 1.27 1.27)
+				)
+				(hide yes)
+			)
+		)
+		(property "Datasheet" ""
+			(at 71.12 72.39 0)
+			(effects
+				(font
+					(size 1.27 1.27)
+				)
+				(hide yes)
+			)
+		)
+		(property "Description" "Power symbol creates a global label with name \"+3.3V\""
+			(at 71.12 72.39 0)
+			(effects
+				(font
+					(size 1.27 1.27)
+				)
+				(hide yes)
+			)
+		)
+		(pin "1"
+		)
+		(instances
+			(project "ESP32_Tracker"
+				(path "/92195c42-0bc4-473e-a890-6f85786d3c69/df595db4-adad-4efb-b42f-768fb30b12a2"
+					(reference "#PWR04")
+					(unit 1)
+				)
+			)
+		)
+	)
+	(symbol
 		(lib_id "Device:C")
 		(at 168.91 59.69 0)
@@
 		(on_board yes)
 		(dnp no)
-		(fields_autoplaced yes)
 		(property "Reference" "#PWR030"
 			(at 96.52 57.15 0)
@@
 		)
 		(property "Value" "+3.3V"
-			(at 96.52 48.26 0)
-			(effects
-				(font
+			(at 96.52 49.276 0)
+			(effects
+				(font

Commit message: modified and labeled layout
Parts:
- added C23: 0.1u, Capacitor_SMD:C_0805_2012Metric, symbol Device:C
Connections:
- net +3.3V: now also C23.1
- net GND: now also C23.2
Other:
- moved on the sheet: C17, C18
Changed lines of the file:
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@@
+	)
+	(junction
+		(at 171.45 64.77)
+		(diameter 0)
+		(color 0 0 0 0)
 	)
 	(junction
@@
 	)
 	(junction
+		(at 182.88 54.61)
+		(diameter 0)
+		(color 0 0 0 0)
+	)
+	(junction
 		(at 214.63 73.66)
 		(diameter 0)
@@
 	)
 	(junction
-		(at 181.61 54.61)
+		(at 171.45 54.61)
 		(diameter 0)
 		(color 0 0 0 0)
@@
 	)
 	(junction
-		(at 168.91 64.77)
+		(at 158.75 64.77)
 		(diameter 0)
 		(color 0 0 0 0)
@@
 	(wire
 		(pts
-			(xy 181.61 64.77) (xy 181.61 63.5)
+			(xy 171.45 64.77) (xy 171.45 63.5)
 		)
 		(stroke
@@
 	(wire
 		(pts
-			(xy 168.91 66.04) (xy 168.91 64.77)
+			(xy 158.75 66.04) (xy 158.75 64.77)
 		)
 		(stroke
@@
 	(wire
 		(pts
-			(xy 181.61 54.61) (xy 181.61 55.88)
-		)
-		(stroke
-			(width 0)
-			(type default)
-		)
-	)
-	(wire
-		(pts
-			(xy 181.61 54.61) (xy 189.23 54.61)
+			(xy 171.45 54.61) (xy 171.45 55.88)
+		)
+		(stroke
+			(width 0)
+			(type default)
+		)
+	)
+	(wire
+		(pts
+			(xy 171.45 54.61) (xy 182.88 54.61)
 		)
 		(stroke
@@
 	(wire
 		(pts
-			(xy 168.91 63.5) (xy 168.91 64.77)
+			(xy 158.75 63.5) (xy 158.75 64.77)
 		)
 		(stroke
@@
 	(wire
 		(pts
+			(xy 171.45 64.77) (xy 182.88 64.77)
+		)
+		(stroke
+			(width 0)
+			(type default)
+		)
+	)
+	(wire
+		(pts
 			(xy 204.47 86.36) (xy 212.09 86.36)
 		)
@@
 	(wire
 		(pts
+			(xy 182.88 54.61) (xy 189.23 54.61)
+		)
+		(stroke
+			(width 0)
+			(type default)
+		)
+	)
+	(wire
+		(pts
+			(xy 182.88 54.61) (xy 182.88 55.88)
+		)
+		(stroke
+			(width 0)
+			(type default)
+		)
+	)
+	(wire
+		(pts
 			(xy 58.42 82.55) (xy 83.82 82.55)
 		)
@@
 	(wire
 		(pts
-			(xy 168.91 64.77) (xy 181.61 64.77)
+			(xy 182.88 63.5) (xy 182.88 64.77)
+		)
+		(stroke
+			(width 0)
+			(type default)
+		)
+	)
+	(wire
+		(pts
+			(xy 158.75 64.77) (xy 171.45 64.77)
 		)
 		(stroke
@@
 	(wire
 		(pts
-			(xy 181.61 54.61) (xy 168.91 54.61)
+			(xy 171.45 54.61) (xy 158.75 54.61)
 		)
 		(stroke
@@
 	(wire
 		(pts
-			(xy 168.91 54.61) (xy 168.91 55.88)
+			(xy 158.75 54.61) (xy 158.75 55.88)
 		)
 		(stroke
@@
 	)
 	(symbol
+		(lib_id "Device:C")
+		(at 182.88 59.69 0)
+		(mirror y)
+		(unit 1)
+		(exclude_from_sim no)
+		(in_bom yes)
+		(on_board yes)
+		(dnp no)
+		(property "Reference" "C23"
+			(at 179.07 58.4199 0)
+			(effects
+				(font
+					(size 1.27 1.27)
+				)
+				(justify left)
+			)
+		)
+		(property "Value" "0.1u"
+			(at 179.07 60.9599 0)
+			(effects
+				(font
+					(size 1.27 1.27)
+				)
+				(justify left)
+			)
+		)
+		(property "Footprint" "Capacitor_SMD:C_0805_2012Metric"
+			(at 181.9148 63.5 0)
+			(effects
+				(font
+					(size 1.27 1.27)
+				)
+				(hide yes)
+			)
+		)
+		(property "Datasheet" "https://www.lcsc.com/datasheet/C519980.pdf"
+			(at 182.88 59.69 0)
+			(effects
+				(font
+					(size 1.27 1.27)
+				)
+				(hide yes)
+			)
+		)
+		(property "Description" "Unpolarized capacitor"
+			(at 182.88 59.69 0)
+			(effects
+				(font
+					(size 1.27 1.27)
+				)
+				(hide yes)
+			)
+		)
+		(property "LCSC" "C519980"
+			(at 182.88 59.69 0)
+			(effects
+				(font
+					(size 1.27 1.27)
+				)
+				(hide yes)
+			)
+		)
+		(property "MPN" "CC0805KRX7R7BB104"
+			(at 182.88 59.69 0)
+			(effects
+				(font
+					(size 1.27 1.27)
+				)
+				(hide yes)
+			)
+		)
+		(property "Manufacturer" "YAGEO"
+			(at 182.88 59.69 0)
+			(effects
+				(font
+					(size 1.27 1.27)
+				)
+				(hide yes)
+			)
+		)
+		(property "Distributor Link" "https://www.lcsc.com/product-detail/C519980.html"
+			(at 182.88 59.69 0)
+			(effects
+				(font
+					(size 1.27 1.27)
+				)
+				(hide yes)
+			)
+		)
+		(pin "2"
+		)
+		(pin "1"
+		)
+		(instances
+			(project "ESP32_Tracker"
+				(path "/92195c42-0bc4-473e-a890-6f85786d3c69/df595db4-adad-4efb-b42f-768fb30b12a2"
+					(reference "C23")
+					(unit 1)
+				)
+			)
+		)
+	)
+	(symbol
 		(lib_id "Sensor_Magnetic:LIS2MDL")
 		(at 96.52 82.55 0)
@@
 	(symbol
 		(lib_id "Device:C")
-		(at 168.91 59.69 0)
+		(at 158.75 59.69 0)
 		(mirror y)
 		(unit 1)
@@
 		(dnp no)
 		(property "Reference" "C17"
-			(at 165.1 58.4199 0)
+			(at 154.94 58.4199 0)
 			(effects
 				(font
@@
 		)
 		(property "Value" "10u"
-			(at 165.1 60.9599 0)
+			(at 154.94 60.9599 0)
 			(effects
 				(font
@@
 		)
 		(property "Footprint" "Capacitor_SMD:C_0805_2012Metric"
-			(at 167.9448 63.5 0)
+			(at 157.7848 63.5 0)
 			(effects
 				(font
@@
 		)
 		(property "Datasheet" "https://www.lcsc.com/datasheet/C95841.pdf"
-			(at 168.91 59.69 0)
+			(at 158.75 59.69 0)
 			(effects
 				(font
@@
 		)
 		(property "Description" "Unpolarized capacitor"
-			(at 168.91 59.69 0)
+			(at 158.75 59.69 0)
 			(effects
 				(font
@@
 		)
 		(property "LCSC" "C95841"
-			(at 168.91 59.69 0)
+			(at 158.75 59.69 0)
 			(effects
 				(font
@@
 		)
 		(property "MPN" "CL21B106KOQNNNE"
-			(at 168.91 59.69 0)
+			(at 158.75 59.69 0)
 			(effects
 				(font
@@
 		)
 		(property "Manufacturer" "Samsung Electro-Mechanics"
-			(at 168.91 59.69 0)
+			(at 158.75 59.69 0)
 			(effects
 				(font
@@
 		)
 		(property "Distributor Link" "https://www.lcsc.com/product-detail/C95841.html"
-			(at 168.91 59.69 0)
+			(at 158.75 59.69 0)
 			(effects
 				(font
@@
 	(symbol
 		(lib_id "power:GND")
-		(at 168.91 66.04 0)
+		(at 158.75 66.04 0)
 		(unit 1)
 		(exclude_from_sim no)
@@
 		(fields_autoplaced yes)
 		(property "Reference" "#PWR032"
-			(at 168.91 72.39 0)
+			(at 158.75 72.39 0)
 			(effects
 				(font
@@
 		)
 		(property "Value" "GND"
-			(at 168.91 71.12 0)
+			(at 158.75 71.12 0)
 			(effects
 				(font
@@
 		)
 		(property "Footprint" ""
-			(at 168.91 66.04 0)
+			(at 158.75 66.04 0)
 			(effects
 				(font
@@
 		)
 		(property "Datasheet" ""
-			(at 168.91 66.04 0)
+			(at 158.75 66.04 0)
 			(effects
 				(font
@@
 		)
 		(property "Description" "Power symbol creates a global label with name \"GND\" , ground"
-			(at 168.91 66.04 0)
+			(at 158.75 66.04 0)
 			(effects
 				(font
@@
 	(symbol
 		(lib_id "Device:C")
-		(at 181.61 59.69 0)
+		(at 171.45 59.69 0)
 		(mirror y)
 		(unit 1)
@@
 		(dnp no)
 		(property "Reference" "C18"
-			(at 177.8 58.4199 0)
+			(at 167.64 58.4199 0)
 			(effects
 				(font
@@
 		)
 		(property "Value" "0.1u"
-			(at 177.8 60.9599 0)
+			(at 167.64 60.9599 0)
 			(effects
 				(font
@@
 		)
 		(property "Footprint" "Capacitor_SMD:C_0805_2012Metric"
-			(at 180.6448 63.5 0)
+			(at 170.4848 63.5 0)
 			(effects
 				(font
@@
 		)
 		(property "Datasheet" "https://www.lcsc.com/datasheet/C519980.pdf"
-			(at 181.61 59.69 0)
+			(at 171.45 59.69 0)
 			(effects
 				(font
@@
 		)
 		(property "Description" "Unpolarized capacitor"
-			(at 181.61 59.69 0)
+			(at 171.45 59.69 0)
 			(effects
 				(font
@@
 		)
 		(property "LCSC" "C519980"
-			(at 181.61 59.69 0)
+			(at 171.45 59.69 0)
 			(effects
 				(font
@@
 		)
 		(property "MPN" "CC0805KRX7R7BB104"
-			(at 181.61 59.69 0)
+			(at 171.45 59.69 0)
 			(effects
 				(font
@@
 		)
 		(property "Manufacturer" "YAGEO"
-			(at 181.61 59.69 0)
+			(at 171.45 59.69 0)
 			(effects
 				(font
@@
 		)
 		(property "Distributor Link" "https://www.lcsc.com/product-detail/C519980.html"
-			(at 181.61 59.69 0)
-			(effects
-				(font
+			(at 171.45 59.69 0)
+			(effects
+				(font
